Commit message: modified launch files and modesl for testing alternative gazebo plugin libraries

File: ego_gz_bridge/simulation/models/component_snippets.xacro (robot description, xacro)
@@ -260,7 +260,8 @@
   <!-- ================== MAVLINK INTERFACE MACRO ==================== -->
   <!-- =============================================================== -->
+  <!-- Macro to add the mavlink interface. -->
   <xacro:macro name="mavlink_interface_macro"
     params="namespace imu_sub_topic
-      mavlink_sub_topic mavlink_pub_topic mavlink_addr mavlink_tcp_port mavlink_udp_port
+      mavlink_sub_topic mavlink_pub_topic mavlink_addr mavlink_udp_port serial_enabled
       motors_speeds_pub_topic gps_update_freq rotor_count
       reference_magnetic_field_north reference_magnetic_field_east reference_magnetic_field_down
@@ -272,5 +273,5 @@
         <mavlink_addr>$(arg mavlink_addr)</mavlink_addr>
         <mavlink_udp_port>$(arg mavlink_udp_port)</mavlink_udp_port>
-        <mavlink_tcp_port>$(arg mavlink_tcp_port)</mavlink_tcp_port>
+        <serialEnabled>$(arg serial_enabled)</serialEnabled>
         <motorSpeedCommandPubTopic>/gazebo/command/motor_speed</motorSpeedCommandPubTopic>
         <mavlinkControlSubTopic>${mavlink_sub_topic}</mavlinkControlSubTopic>
@@ -293,4 +294,111 @@
     </gazebo>
   </xacro:macro>
+  <!-- <xacro:macro name="mavlink_interface_macro" params="namespace imu_sub_topic mavlink_addr mavlink_udp_port">
+    <gazebo>
+      <plugin name="mavlink_interface" filename="librotors_gazebo_mavlink_interface.so">
+        <robotNamespace>${namespace}</robotNamespace>
+        <imuSubTopic>${imu_sub_topic}</imuSubTopic>
+        <mavlink_addr>$(arg mavlink_addr)</mavlink_addr>
+        <mavlink_udp_port>$(arg mavlink_udp_port)</mavlink_udp_port>
+        <motorSpeedCommandPubTopic>/gazebo/command/motor_speed</motorSpeedCommandPubTopic>
+        <control_channels>
+          <channel name="rotor1">
+            <input_index>0</input_index>
+            <input_offset>0</input_offset>
+            <input_scaling>1000</input_scaling>
+            <zero_position_disarmed>0</zero_position_disarmed>
+            <zero_position_armed>100</zero_position_armed>
+            <joint_control_type>velocity</joint_control_type>
+          </channel>
+          <channel name="rotor2">
+            <input_index>1</input_index>
+            <input_offset>0</input_offset>
+            <input_scaling>1000</input_scaling>
+            <zero_position_disarmed>0</zero_position_disarmed>
+            <zero_position_armed>100</zero_position_armed>
+            <joint_control_type>velocity</joint_control_type>
+          </channel>
+          <channel name="rotor3">
+            <input_index>2</input_index>
+            <input_offset>0</input_offset>
+            <input_scaling>1000</input_scaling>
+            <zero_position_disarmed>0</zero_position_disarmed>
+            <zero_position_armed>100</zero_position_armed>
+            <joint_control_type>velocity</joint_control_type>
+          </channel>
+          <channel name="rotor4">
+            <input_index>3</input_index>
+            <input_offset>0</input_offset>
+            <input_scaling>1000</input_scaling>
+            <zero_position_disarmed>0</zero_position_disarmed>
+            <zero_position_armed>100</zero_position_armed>
+            <joint_control_type>velocity</joint_control_type>
+          </channel>
+          <channel name="rotor5">
+            <input_index>4</input_index>
+            <input_offset>1</input_offset>
+            <input_scaling>324.6</input_scaling>
+            <zero_position_disarmed>0</zero_position_disarmed>
+            <zero_position_armed>0</zero_position_armed>
+            <joint_control_type>velocity</joint_control_type>
+            <joint_control_pid>
+              <p>0.1</p>
+              <i>0</i>
+              <d>0</d>
+              <iMax>0.0</iMax>
+              <iMin>0.0</iMin>
+              <cmdMax>2</cmdMax>
+              <cmdMin>-2</cmdMin>
+            </joint_control_pid>
+            <joint_name>zephyr_delta_wing::propeller_joint</joint_name>
+          </channel>
+          <channel name="rotor6">
+            <input_index>5</input_index>
+            <input_offset>0</input_offset>
+            <input_scaling>0.524</input_scaling>
+            <zero_position_disarmed>0</zero_position_disarmed>
+            <zero_position_armed>0</zero_position_armed>
+            <joint_control_type>position</joint_control_type>
+            <joint_name>zephyr_delta_wing::flap_left_joint</joint_name>
+            <joint_control_pid>
+              <p>10.0</p>
+              <i>0</i>
+              <d>0</d>
+              <iMax>0</iMax>
+              <iMin>0</iMin>
+              <cmdMax>20</cmdMax>
+              <cmdMin>-20</cmdMin>
+            </joint_control_pid>
+          </channel>
+          <channel name="rotor7">
+            <input_index>6</input_index>
+            <input_offset>0</input_offset>
+            <input_scaling>0.524</input_scaling>
+            <zero_position_disarmed>0</zero_position_disarmed>
+            <zero_position_armed>0</zero_position_armed>
+            <joint_control_type>position</joint_control_type>
+            <joint_name>zephyr_delta_wing::flap_right_joint</joint_name>
+            <joint_control_pid>
+              <p>10.0</p>
+              <i>0</i>
+              <d>0</d>
+              <iMax>0</iMax>
+              <iMin>0</iMin>
+              <cmdMax>20</cmdMax>
+              <cmdMin>-20</cmdMin>
+            </joint_control_pid>
+          </channel>
+          <channel name="rotor8">
+            <input_index>7</input_index>
+            <input_offset>0</input_offset>
+            <input_scaling>0.524</input_scaling>
+            <zero_position_disarmed>0</zero_position_disarmed>
+            <zero_position_armed>0</zero_position_armed>
+            <joint_control_type>position</joint_control_type>
+          </channel>
+        </control_channels>
+      </plugin>
+    </gazebo>
+  </xacro:macro> -->
   <!-- Macro to add an IMU. -->
   <xacro:macro name="imu_plugin_macro"
@@ -888,6 +996,6 @@
       mavlink_sub_topic="/mavlink/from"
       imu_sub_topic="${imu_sub_topic}"
+      serial_enabled="false"
       mavlink_addr="INADDR_ANY"
-      mavlink_tcp_port="4560"
       mavlink_udp_port="14560"
       mavlink_pub_topic="/mavlink/to"

File: ego_gz_bridge/simulation/models/hummingbird_base.xacro (robot description, xacro)
@@ -17,4 +17,11 @@
 -->
 <robot name="hummingbird" xmlns:xacro="http://ros.org/wiki/xacro">
+  <!-- Properties that can be assigned at build time as arguments.
+  Is there a reason not to make all properties arguments?
+  -->
+  <xacro:arg name='mavlink_addr' default='INADDR_ANY' />
+  <xacro:arg name='mavlink_udp_port' default='14560' />
+  <xacro:arg name='visual_material' default='DarkGrey' />
+  <xacro:arg name='serial_enabled' default='false' />
   <xacro:include filename="$(find ego_gz_bridge)/simulation/models/component_snippets.xacro" />
   <!-- Instantiate hummingbird "mechanics" -->
@@ -24,5 +31,6 @@
   <xacro:if value="$(arg enable_mavlink_interface)">
     <!-- Instantiate mavlink telemetry interface. -->
-    <xacro:default_mavlink_interface namespace="${namespace}" imu_sub_topic="imu" rotor_count="4" />
+    <xacro:default_mavlink_interface
+      namespace="${namespace}" imu_sub_topic="imu" rotor_count="4" />
   </xacro:if>
   <!-- Mount an ADIS16448 IMU. -->

File: ego_gz_bridge/simulation/models/iris_pro/iris_pro.gazebo.xacro (robot description, xacro)
@@ -4,4 +4,5 @@
   <xacro:arg name="camera_visual" default="false"/>
   <xacro:arg name="imu_visual"    default="false"/> -->
+  <xacro:arg name="namespace"  default="iris"/>
   <gazebo reference="base_link">
     <material>Gazebo/DarkGrey</material>
@@ -134,6 +135,6 @@
     </plugin>
   </gazebo>
-  <!-- ///// Sensors ///// -->
-  <gazebo reference="gps_link">
+  <!-- ///// GPS ///// -->
+  <!-- <gazebo reference="gps_link">
     <material>Gazebo/FlatBlack</material>
     <sensor name="gps_link" type="gps">
@@ -153,5 +154,18 @@
       </plugin>
     </sensor>
-  </gazebo>
+  </gazebo> -->
+  <gazebo>
+    <plugin name="gps_plugin" filename="libgazebo_gps_plugin.so">
+      <robotNamespace/>
+      <gpsNoise>true</gpsNoise>
+      <gpsXYRandomWalk>2.0</gpsXYRandomWalk>
+      <gpsZRandomWalk>4.0</gpsZRandomWalk>
+      <gpsXYNoiseDensity>2.0e-4</gpsXYNoiseDensity>
+      <gpsZNoiseDensity>4.0e-4</gpsZNoiseDensity>
+      <gpsVXYNoiseDensity>0.2</gpsVXYNoiseDensity>
+      <gpsVZNoiseDensity>0.4</gpsVZNoiseDensity>
+    </plugin>
+  </gazebo>
+  <!-- ///// Ground truth ///// -->
   <gazebo>
     <plugin name='groundtruth_plugin' filename='libgazebo_groundtruth_plugin.so'>
@@ -159,4 +173,5 @@
     </plugin>
   </gazebo>
+  <!-- ///// Magnetometer ///// -->
   <gazebo>
     <plugin name='magnetometer_plugin' filename='libgazebo_magnetometer_plugin.so'>
@@ -169,4 +184,5 @@
     </plugin>
   </gazebo>
+  <!-- ///// Barometer ///// -->
   <gazebo>
     <plugin name='barometer_plugin' filename='libgazebo_barometer_plugin.so'>
@@ -177,129 +193,8 @@
     </plugin>
   </gazebo>
-  <gazebo>
-    <plugin name='mavlink_interface' filename='libgazebo_mavlink_interface.so'>
-      <robotNamespace/>
-      <imuSubTopic>/imu</imuSubTopic>
-      <magSubTopic>/mag</magSubTopic>
-      <gpsSubTopic>/gps</gpsSubTopic>
-      <baroSubTopic>/baro</baroSubTopic>
-      <mavlink_addr>INADDR_ANY</mavlink_addr>
-      <mavlink_tcp_port>4560</mavlink_tcp_port>
-      <mavlink_udp_port>14560</mavlink_udp_port>
-      <serialEnabled>0</serialEnabled>
-      <serialDevice>/dev/ttyACM0</serialDevice>
-      <baudRate>921600</baudRate>
-      <qgc_addr>INADDR_ANY</qgc_addr>
-      <qgc_udp_port>14550</qgc_udp_port>
-      <sdk_addr>INADDR_ANY</sdk_addr>
-      <sdk_udp_port>14540</sdk_udp_port>
-      <hil_mode>0</hil_mode>
-      <hil_state_level>0</hil_state_level>
-      <send_vision_estimation>0</send_vision_estimation>
-      <send_odometry>1</send_odometry>
-      <enable_lockstep>1</enable_lockstep>
-      <use_tcp>1</use_tcp>
-      <motorSpeedCommandPubTopic>/gazebo/command/motor_speed</motorSpeedCommandPubTopic>
-      <control_channels>
-        <channel name='rotor1'>
-          <input_index>0</input_index>
-          <input_offset>0</input_offset>
-          <input_scaling>1000</input_scaling>
-          <zero_position_disarmed>0</zero_position_disarmed>
-          <zero_position_armed>100</zero_position_armed>
-          <joint_control_type>velocity</joint_control_type>
-        </channel>
-        <channel name='rotor2'>
-          <input_index>1</input_index>
-          <input_offset>0</input_offset>
-          <input_scaling>1000</input_scaling>
-          <zero_position_disarmed>0</zero_position_disarmed>
-          <zero_position_armed>100</zero_position_armed>
-          <joint_control_type>velocity</joint_control_type>
-        </channel>
-        <channel name='rotor3'>
-          <input_index>2</input_index>
-          <input_offset>0</input_offset>
-          <input_scaling>1000</input_scaling>
-          <zero_position_disarmed>0</zero_position_disarmed>
-          <zero_position_armed>100</zero_position_armed>
-          <joint_control_type>velocity</joint_control_type>
-        </channel>
-        <channel name='rotor4'>
-          <input_index>3</input_index>
-          <input_offset>0</input_offset>
-          <input_scaling>1000</input_scaling>
-          <zero_position_disarmed>0</zero_position_disarmed>
-          <zero_position_armed>100</zero_position_armed>
-          <joint_control_type>velocity</joint_control_type>
-        </channel>
-        <channel name='rotor5'>
-          <input_index>4</input_index>
-          <input_offset>1</input_offset>
-          <input_scaling>324.6</input_scaling>
-          <zero_position_disarmed>0</zero_position_disarmed>
-          <zero_position_armed>0</zero_position_armed>
-          <joint_control_type>velocity</joint_control_type>
-          <joint_control_pid>
-            <p>0.1</p>
-            <i>0</i>
-            <d>0</d>
-            <iMax>0.0</iMax>
-            <iMin>0.0</iMin>
-            <cmdMax>2</cmdMax>
-            <cmdMin>-2</cmdMin>
-          </joint_control_pid>
-          <joint_name>zephyr_delta_wing::propeller_joint</joint_name>
-        </channel>
-        <channel name='rotor6'>
-          <input_index>5</input_index>
-          <input_offset>0</input_offset>
-          <input_scaling>0.524</input_scaling>
-          <zero_position_disarmed>0</zero_position_disarmed>
-          <zero_position_armed>0</zero_position_armed>
-          <joint_control_type>position</joint_control_type>
-          <joint_name>zephyr_delta_wing::flap_left_joint</joint_name>
-          <joint_control_pid>
-            <p>10.0</p>
-            <i>0</i>
-            <d>0</d>
-            <iMax>0</iMax>
-            <iMin>0</iMin>
-            <cmdMax>20</cmdMax>
-            <cmdMin>-20</cmdMin>
-          </joint_control_pid>
-        </channel>
-        <channel name='rotor7'>
-          <input_index>6</input_index>
-          <input_offset>0</input_offset>
-          <input_scaling>0.524</input_scaling>
-          <zero_position_disarmed>0</zero_position_disarmed>
-          <zero_position_armed>0</zero_position_armed>
-          <joint_control_type>position</joint_control_type>
-          <joint_name>zephyr_delta_wing::flap_right_joint</joint_name>
-          <joint_control_pid>
-            <p>10.0</p>
-            <i>0</i>
-            <d>0</d>
-            <iMax>0</iMax>
-            <iMin>0</iMin>
-            <cmdMax>20</cmdMax>
-            <cmdMin>-20</cmdMin>
-          </joint_control_pid>
-        </channel>
-        <channel name='rotor8'>
-          <input_index>7</input_index>
-          <input_offset>0</input_offset>
-          <input_scaling>0.524</input_scaling>
-          <zero_position_disarmed>0</zero_position_disarmed>
-          <zero_position_armed>0</zero_position_armed>
-          <joint_control_type>position</joint_control_type>
-        </channel>
-      </control_channels>
-    </plugin>
-  </gazebo>
-  <gazebo reference="imu_link">
-    <plugin name='rotors_gazebo_imu_plugin' filename='libgazebo_imu_plugin.so'>
-      <robotNamespace/>
+  <!-- ///// IMU Link ///// -->
+  <!-- <gazebo>
+    <plugin name='gazebo_imu_plugin' filename='libgazebo_imu_plugin.so'>
+      <robotNamespace></robotNamespace>
       <linkName>/imu_link</linkName>
       <imuTopic>/imu</imuTopic>
@@ -313,39 +208,151 @@
       <accelerometerTurnOnBiasSigma>0.196</accelerometerTurnOnBiasSigma>
     </plugin>
-  </gazebo>
-  <gazebo>
+  </gazebo> -->
+  <!-- <gazebo>
     <plugin name='gps_plugin' filename='libgazebo_gps_plugin.so'>
       <robotNamespace/>
       <gpsNoise>1</gpsNoise>
     </plugin>
-  </gazebo>
+  </gazebo> -->
+  <!-- Default gazebo IMU -->
   <!-- <gazebo>
     <plugin name="imu_plugin" filename="libgazebo_ros_imu.so">
+      <robotNamespace></robotNamespace>
       <alwaysOn>true</alwaysOn>
       <bodyName>imu_link</bodyName>
       <frameName>imu_link</frameName>
       <topicName>imu</topicName>
-      <serviceName>imu_service</serviceName>
+      <serviceName>imu/service</serviceName>
       <gaussianNoise>0.0</gaussianNoise>
-      <updateRate>0</updateRate>
-      <imu>
-        <noise>
-          <type>gaussian</type>
-          <rate>
-            <mean>0.0</mean>
-            <stddev>2e-4</stddev>
-            <bias_mean>0.0000075</bias_mean>
-            <bias_stddev>0.0000008</bias_stddev>
-          </rate>
-          <accel>
-            <mean>0.0</mean>
-            <stddev>1.7e-2</stddev>
-            <bias_mean>0.1</bias_mean>
-            <bias_stddev>0.001</bias_stddev>
-          </accel>
-        </noise>
-      </imu>
+      <updateRate>10.0</updateRate>
+      <rpyOffsets>0 0 0</rpyOffsets>
     </plugin>
   </gazebo> -->
   <!-- ///// Camera ///// -->
+  <!-- ///// Mavlink interface ///// -->
+    <gazebo>
+      <plugin name="mavlink_interface" filename="libgazebo_mavlink_interface.so">
+        <robotNamespace></robotNamespace>
+        <imuSubTopic>/imu</imuSubTopic>
+        <gpsSubTopic>/gps</gpsSubTopic>
+        <magSubTopic>/mag</magSubTopic>
+        <baroSubTopic>/baro</baroSubTopic>
+        <mavlink_addr>INADDR_ANY</mavlink_addr>
+        <mavlink_udp_port>14560</mavlink_udp_port>
+        <mavlink_tcp_port>4560</mavlink_tcp_port>
+        <serialEnabled>0</serialEnabled>
+        <serialDevice>/dev/ttyACM0</serialDevice>
+        <baudRate>921600</baudRate>
+        <qgc_addr>INADDR_ANY</qgc_addr>
+        <qgc_udp_port>14550</qgc_udp_port>
+        <sdk_addr>INADDR_ANY</sdk_addr>
+        <sdk_udp_port>14540</sdk_udp_port>
+        <hil_mode>0</hil_mode>
+        <hil_state_level>0</hil_state_level>
+        <vehicle_is_tailsitter>false</vehicle_is_tailsitter>
+        <send_vision_estimation>0</send_vision_estimation>
+        <send_odometry>1</send_odometry>
+        <enable_lockstep>1</enable_lockstep>
+        <use_tcp>1</use_tcp>
+        <motorSpeedCommandPubTopic>/gazebo/command/motor_speed</motorSpeedCommandPubTopic>
+        <control_channels>
+          <channel name="rotor1">
+            <input_index>0</input_index>
+            <input_offset>0</input_offset>
+            <input_scaling>1000</input_scaling>
+            <zero_position_disarmed>0</zero_position_disarmed>
+            <zero_position_armed>100</zero_position_armed>
+            <joint_control_type>velocity</joint_control_type>
+          </channel>
+          <channel name="rotor2">
+            <input_index>1</input_index>
+            <input_offset>0</input_offset>
+            <input_scaling>1000</input_scaling>
+            <zero_position_disarmed>0</zero_position_disarmed>
+            <zero_position_armed>100</zero_position_armed>
+            <joint_control_type>velocity</joint_control_type>
+          </channel>
+          <channel name="rotor3">
+            <input_index>2</input_index>
+            <input_offset>0</input_offset>
+            <input_scaling>1000</input_scaling>
+            <zero_position_disarmed>0</zero_position_disarmed>
+            <zero_position_armed>100</zero_position_armed>
+            <joint_control_type>velocity</joint_control_type>
+          </channel>
+          <channel name="rotor4">
+            <input_index>3</input_index>
+            <input_offset>0</input_offset>
+            <input_scaling>1000</input_scaling>
+            <zero_position_disarmed>0</zero_position_disarmed>
+            <zero_position_armed>100</zero_position_armed>
+            <joint_control_type>velocity</joint_control_type>
+          </channel>
+          <channel name="rotor5">
+            <input_index>4</input_index>
+            <input_offset>1</input_offset>
+            <input_scaling>324.6</input_scaling>
+            <zero_position_disarmed>0</zero_position_disarmed>
+            <zero_position_armed>0</zero_position_armed>
+            <joint_control_type>velocity</joint_control_type>
+            <joint_control_pid>
+              <p>0.1</p>
+              <i>0</i>
+              <d>0</d>
+              <iMax>0.0</iMax>
+              <iMin>0.0</iMin>
+              <cmdMax>2</cmdMax>
+              <cmdMin>-2</cmdMin>
+            </joint_control_pid>
+            <joint_name>zephyr_delta_wing::propeller_joint</joint_name>
+          </channel>
+          <channel name="rotor6">
+            <input_index>5</input_index>
+            <input_offset>0</input_offset>
+            <!-- joint limits [-0.524, 0.524] -->
+            <input_scaling>0.524</input_scaling>
+            <zero_position_disarmed>0</zero_position_disarmed>
+            <zero_position_armed>0</zero_position_armed>
+            <joint_control_type>position</joint_control_type>
+            <joint_name>zephyr_delta_wing::flap_left_joint</joint_name>
+            <joint_control_pid>
+              <p>10.0</p>
+              <i>0</i>
+              <d>0</d>
+              <iMax>0</iMax>
+              <iMin>0</iMin>
+              <cmdMax>20</cmdMax>
+              <cmdMin>-20</cmdMin>
+            </joint_control_pid>
+          </channel>
+          <channel name="rotor7">
+            <input_index>6</input_index>
+            <input_offset>0</input_offset>
+            <!-- joint limits [-0.524, 0.524] -->
+            <input_scaling>0.524</input_scaling>
+            <zero_position_disarmed>0</zero_position_disarmed>
+            <zero_position_armed>0</zero_position_armed>
+            <joint_control_type>position</joint_control_type>
+            <joint_name>zephyr_delta_wing::flap_right_joint</joint_name>
+            <joint_control_pid>
+              <p>10.0</p>
+              <i>0</i>
+              <d>0</d>
+              <iMax>0</iMax>
+              <iMin>0</iMin>
+              <cmdMax>20</cmdMax>
+              <cmdMin>-20</cmdMin>
+            </joint_control_pid>
+          </channel>
+          <channel name="rotor8">
+            <input_index>7</input_index>
+            <input_offset>0</input_offset>
+            <input_scaling>0.524</input_scaling>
+            <zero_position_disarmed>0</zero_position_disarmed>
+            <zero_position_armed>0</zero_position_armed>
+            <joint_control_type>position</joint_control_type>
+          </channel>
+        </control_channels>
+      </plugin>
+    </gazebo>
 </robot>

File: ego_gz_bridge/simulation/models/iris_pro/iris_pro.urdf.xacro (robot description, xacro)
@@ -1,4 +1,4 @@
 <?xml version="1.0" ?>
-<robot name="turtlebot3_waffle" xmlns:xacro="http://ros.org/wiki/xacro">
+<robot name="iris_pro" xmlns:xacro="http://ros.org/wiki/xacro">
   <xacro:include filename="$(find ego_gz_bridge)/simulation/models/iris_pro/common_properties.xacro"/>
   <xacro:include filename="$(find ego_gz_bridge)/simulation/models/iris_pro/iris_pro.gazebo.xacro"/>
@@ -30,5 +30,5 @@
     </inertial>
   </link>
-  <link name="imu_link">
+  <link name="/imu_link">
     <inertial>
       <origin xyz="0 0 0" rpy="0 0 0"/>
@@ -176,5 +176,5 @@
     <origin xyz="0 0 0" rpy="0 0 0"/>
     <parent link="base_link"/>
-    <child link="imu_link"/>
+    <child link="/imu_link"/>
   </joint>
   <joint name='gps_joint' type='fixed'>
